File: pcb/null-city-badge.kicad_sch (KiCad schematic)
At the start: 81 parts, among them J1 USB_C_Receptacle_USB2.0_16P, J10 Conn_01x10_Pin, J2 Conn_01x02_Pin, J3 Conn_01x06_Pin, J4 Conn_01x24_Socket, J8 Conn_01x06_Pin, Q1 SS8050, Q2 SS8050, Q3 IRLML0030, Q4 AO3401A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

Commit message: feat: improve pinout and remove sdcard and lora module, update design
Parts:
- removed J3: Conn_01x06_Pin, Connector_PinHeader_2.54mm:PinHeader_1x06_P2.54mm_Vertical, symbol Connector:Conn_01x06_Pin
- removed R11, R12: 2K2, Resistor_SMD:R_0402_1005Metric, symbol Device:R
- removed R19, R8: 10K, Resistor_SMD:R_0402_1005Metric, symbol Device:R
- removed U2: CP2102N-Axx-xQFN28, Package_DFN_QFN:QFN-28-1EP_5x5mm_P0.5mm_EP3.35x3.35mm, symbol Interface_USB:CP2102N-Axx-xQFN28
- removed U3: SE050C2HQ1_Z01SDZ, NIP_MOD:QFN40P300X300X33-21N, symbol PCM_NIP_MOD:SE050C2HQ1_Z01SDZ
- added J3: Conn_01x04_Pin, Connector_PinHeader_2.54mm:PinHeader_1x04_P2.54mm_Vertical, symbol Connector:Conn_01x04_Pin
- added U15: CH340C, Package_SO:SOIC-16_3.9x9.9mm_P1.27mm, symbol Interface_USB:CH340C
- added U16: ATECC608B-SSHDA, Package_SO:SOIC-8_3.9x4.9mm_P1.27mm, symbol Security:ATECC608B-SSHDA
- J2: footprint Connector_JST:JST_PH_S2B-PH-SM4-TB_1x02-1MP_P2.00mm_Horizontal -> Connector_JST:JST_GH_SM02B-GHS-TB_1x02-1MP_P1.25mm_Horizontal
Connections:
- net 1CS: now also J3.3 (Pin_3)
- net 1SCK: now also J10.4 (Pin_4)
- net 1SDI: now also J10.3 (Pin_3)
- net 1SDO: now also J3.4 (Pin_4)
- net 3V3: now also C2.1, C3.1, C9.1, U15.16 (VCC), U15.4 (V3), U16.8 (VCC)
- net D+: now also U15.5 (UD+)
- net D-: now also U15.6 (UD-)
- net DTR: now also U15.13 (~{DTR})
- net GND1: now also J3.1 (Pin_1), U15.1 (GND), U16.4 (GND)
- net RTS: now also U15.14 (~{RTS})
- net SCK: no longer J10.4 (Pin_4)
- net SCL: now also U16.6 (SCL)
- net SDA: now also U16.5 (SDA)
- net SDI: no longer J10.3 (Pin_3)
- net TX0: now also U15.3 (RXD)
- net VBUS: now also C1.1; no longer C2.1, C3.1
- net VSYS: now also J3.2 (Pin_2)
- net at R1.1: now also U15.2 (TXD)
Other:
- removed sheet LORA MODULE
- removed sheet SD CARD MODULE
- moved on the sheet: BOOT1, C1, C10, C11, C12, C13, C14, C15, C16, C17, C18, C19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

Commit message: fix sub ghz, epaper and audio module
Parts:
- added R8: 56K, Resistor_SMD:R_0402_1005Metric, symbol Device:R
Connections:
- net 3V3: now also J4.10 (Pin_10), J4.9 (Pin_9); no longer J4.15 (Pin_15), J4.16 (Pin_16)
- net BUSY: now also J4.16 (Pin_16), U1.23 (IO21); no longer J4.9 (Pin_9), U1.10 (IO17)
- net CS: now also J4.13 (Pin_13), U1.20 (IO12); no longer J4.12 (Pin_12), U1.21 (IO13)
- net DC: now also J4.14 (Pin_14), U1.21 (IO13); no longer J4.11 (Pin_11), U1.20 (IO12)
- net GDR: now also J4.23 (Pin_23), R8.2; no longer J4.2 (Pin_2)
- net GND1: now also J4.17 (Pin_17), R8.1
- net RESE: now also J4.22 (Pin_22); no longer J4.3 (Pin_3)
- net RS: now also J4.15 (Pin_15), U1.22 (IO14); no longer J4.10 (Pin_10), U1.19 (IO11)
- net SCK: now also J4.12 (Pin_12), U1.19 (IO11); no longer J4.13 (Pin_13), U1.22 (IO14)
- net SDI: now also J4.11 (Pin_11), U1.10 (IO17); no longer J4.14 (Pin_14), U1.23 (IO21)
- net VGH: now also J4.4 (Pin_4); no longer J4.21 (Pin_21)
- net VGL: now also J4.2 (Pin_2); no longer J4.23 (Pin_23)
- net at C18.2: now also J4.7 (Pin_7); no longer J4.18 (Pin_18)
- net at C16.2: now also J4.3 (Pin_3); no longer J4.22 (Pin_22)
- net at C17.2: now also J4.5 (Pin_5); no longer J4.20 (Pin_20)
- net at J4.1 (Pin_1): now also C15.2
- net at J4.24 (Pin_24): no longer C15.2
- net at C19.2: now also J4.20 (Pin_20); no longer J4.5 (Pin_5)
Changed lines of the file:
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@@
 	)
 	(junction
+		(at 257.81 140.97)
+		(diameter 0)
+		(color 0 0 0 0)
+	)
+	(junction
 		(at 115.57 120.65)
 		(diameter 0)
@@
 	(wire
 		(pts
+			(xy 180.34 142.24) (xy 189.23 142.24)
+		)
+		(stroke
+			(width 0)
+			(type default)
+		)
+	)
+	(wire
+		(pts
 			(xy 100.33 31.75) (xy 100.33 30.48)
 		)
@@
 	(wire
 		(pts
+			(xy 180.34 149.86) (xy 180.34 142.24)
+		)
+		(stroke
+			(width 0)
+			(type default)
+		)
+	)
+	(wire
+		(pts
 			(xy 33.02 43.18) (xy 35.56 43.18)
 		)
@@
 	(wire
 		(pts
+			(xy 271.78 138.43) (xy 257.81 138.43)
+		)
+		(stroke
+			(width 0)
+			(type default)
+		)
+	)
+	(wire
+		(pts
 			(xy 44.45 83.82) (xy 45.72 83.82)
 		)
@@
 	(wire
 		(pts
+			(xy 257.81 138.43) (xy 257.81 140.97)
+		)
+		(stroke
+			(width 0)
+			(type default)
+		)
+	)
+	(wire
+		(pts
 			(xy 266.7 123.19) (xy 271.78 123.19)
 		)
@@
 	(wire
 		(pts
-			(xy 181.61 142.24) (xy 189.23 142.24)
-		)
-		(stroke
-			(width 0)
-			(type default)
-		)
-	)
-	(wire
-		(pts
 			(xy 184.15 22.86) (xy 184.15 24.13)
 		)
@@
 		)
 	)
+	(label "SCK"
+		(at 157.48 107.95 0)
+		(effects
+			(font
+				(size 1.27 1.27)
+			)
+			(justify left bottom)
+		)
+	)
 	(label "SDA"
 		(at 13.97 130.81 0)
@@
 		)
 	)
-	(label "DC"
-		(at 157.48 110.49 0)
+	(label "RS"
+		(at 157.48 115.57 0)
 		(effects
 			(font
@@
 		)
 	)
-	(label "CS"
-		(at 157.48 113.03 0)
+	(label "SDI"
+		(at 199.39 80.01 180)
 		(effects
 			(font
 				(size 1.27 1.27)
 			)
-			(justify left bottom)
+			(justify right bottom)
 		)
 	)
@@
 		)
 	)
-	(label "RS"
-		(at 157.48 107.95 0)
-		(effects
-			(font
-				(size 1.27 1.27)
-			)
-			(justify left bottom)
-		)
-	)
 	(label "1SCK"
 		(at 250.19 76.2 180)
@@
 		)
 	)
+	(label "SDI"
+		(at 247.65 104.14 180)
+		(effects
+			(font
+				(size 1.27 1.27)
+			)
+			(justify right bottom)
+		)
+	)
 	(label "PWR"
 		(at 200.66 40.64 180)
@@
 		)
 	)
+	(label "CS"
+		(at 157.48 110.49 0)
+		(effects
+			(font
+				(size 1.27 1.27)
+			)
+			(justify left bottom)
+		)
+	)
+	(label "BUSY"
+		(at 199.39 90.17 180)
+		(effects
+			(font
+				(size 1.27 1.27)
+			)
+			(justify right bottom)
+		)
+	)
 	(label "1CS"
 		(at 199.39 105.41 180)
@@
 		)
 	)
+	(label "DC"
+		(at 157.48 113.03 0)
+		(effects
+			(font
+				(size 1.27 1.27)
+			)
+			(justify left bottom)
+		)
+	)
 	(label "VGH"
 		(at 266.7 148.59 0)
@@
 		)
 	)
-	(label "SDI"
-		(at 199.39 90.17 180)
-		(effects
-			(font
-				(size 1.27 1.27)
-			)
-			(justify right bottom)
-		)
-	)
 	(label "3SDI"
 		(at 157.48 97.79 0)
@@
 		)
 	)
-	(label "SCK"
-		(at 157.48 115.57 0)
-		(effects
-			(font
-				(size 1.27 1.27)
-			)
-			(justify left bottom)
-		)
-	)
 	(label "2SDO"
 		(at 278.13 73.66 180)
@@
 		)
 	)
-	(label "BUSY"
-		(at 199.39 80.01 180)
-		(effects
-			(font
-				(size 1.27 1.27)
-			)
-			(justify right bottom)
-		)
-	)
 	(label "PWR"
 		(at 199.39 82.55 180)
@@
 	(symbol
 		(lib_id "power:GND")
+		(at 180.34 157.48 0)
+		(unit 1)
+		(exclude_from_sim no)
+		(in_bom yes)
+		(on_board yes)
+		(dnp no)
+		(fields_autoplaced yes)
+		(property "Reference" "#PWR02"
+			(at 180.34 163.83 0)
+			(effects
+				(font
+					(size 1.27 1.27)
+				)
+				(hide yes)
+			)
+		)
+		(property "Value" "GND1"
+			(at 180.34 162.56 0)
+			(effects
+				(font
+					(size 1.27 1.27)
+				)
+			)
+		)
+		(property "Footprint" ""
+			(at 180.34 157.48 0)
+			(effects
+				(font
+					(size 1.27 1.27)
+				)
+				(hide yes)
+			)
+		)
+		(property "Datasheet" ""
+			(at 180.34 157.48 0)
+			(effects
+				(font
+					(size 1.27 1.27)
+				)
+				(hide yes)
+			)
+		)
+		(property "Description" "Power symbol creates a global label with name \"GND\" , ground"
+			(at 180.34 157.48 0)
+			(effects
+				(font
+					(size 1.27 1.27)
+				)
+				(hide yes)
+			)
+		)
+		(pin "1"
+		)
+		(instances
+			(project "null-city-badge"
+				(path "/96a9ebd7-4f87-4060-87a7-f00d27473ddc"
+					(reference "#PWR02")
+					(unit 1)
+				)
+			)
+		)
+	)
+	(symbol
+		(lib_id "power:GND")
 		(at 227.33 157.48 0)
 		(unit 1)
@@
 	(symbol
 		(lib_id "Connector:Conn_01x24_Socket")
-		(at 276.86 125.73 0)
+		(at 276.86 128.27 0)
+		(mirror x)
 		(unit 1)
 		(exclude_from_sim no)
@@
 		(dnp no)
 		(property "Reference" "J4"
-			(at 281.432 117.348 90)
+			(at 281.432 136.652 90)
 			(effects
 				(font
@@
 		)
 		(property "Value" "Conn_01x24_Socket"
-			(at 278.892 117.348 90)
+			(at 278.892 136.652 90)
 			(effects
 				(font
@@
 		)
 		(property "Footprint" "Connector_FFC-FPC:Hirose_FH12-24S-0.5SH_1x24-1MP_P0.50mm_Horizontal"
-			(at 276.86 125.73 0)
+			(at 276.86 128.27 0)
 			(effects
 				(font
@@
 		)
 		(property "Datasheet" "~"
-			(at 276.86 125.73 0)
+			(at 276.86 128.27 0)
 			(effects
 				(font
@@
 		)
 		(property "Description" "Generic connector, single row, 01x24, script generated"
-			(at 276.86 125.73 0)
+			(at 276.86 128.27 0)
 			(effects
 				(font
@@
 					(unit 1)
 				)
+			)
+		)
+	)
+	(symbol
+		(lib_id "Device:R")
+		(at 180.34 153.67 0)
+		(mirror x)
+		(unit 1)
+		(exclude_from_sim no)
+		(in_bom yes)
+		(on_board yes)
+		(dnp no)
+		(property "Reference" "R8"
+			(at 176.53 152.3999 0)
+			(effects
+				(font
+					(size 1.27 1.27)
+				)
+				(justify right)
+			)
+		)
+		(property "Value" "56K"
+			(at 176.53 154.9399 0)
+			(effects
+				(font
+					(size 1.27 1.27)
+				)
+				(justify right)
+			)
+		)
+		(property "Footprint" "Resistor_SMD:R_0402_1005Metric"
+			(at 178.562 153.67 90)
+			(effects
+				(font
+					(size 1.27 1.27)
+				)
+				(hide yes)
+			)
+		)
+		(property "Datasheet" "~"
+			(at 180.34 153.67 0)
+			(effects
+				(font
+					(size 1.27 1.27)
+				)
+				(hide yes)
+			)
+		)
+		(property "Description" "Resistor"
+			(at 180.34 153.67 0)
+			(effects
+				(font
+					(size 1.27 1.27)
+				)
+				(hide yes)
+			)
+		)
+		(pin "1"
+		)
+		(pin "2"
+		)
+		(instances
+			(project "null-city-badge"
+				(path "/96a9ebd7-4f87-4060-87a7-f00d27473ddc"
+					(reference "R8")
+					(unit 1)
+				)
